File: Kicad/JR-100_SD.kicad_pcb (KiCad board)
At the start: 2 copper layers, 100 x 100 mm, 31 parts, among them J1 Conn_01x25, J2 Conn_01x25, J3 MSX JOY STICK, J4 IN 5V, J5 EXT 5V, J6 Micro_SD_Card_Kit, J7 MicroSD Card Adapter, J8 Conn_01x01, SW1 SW_Push, U1 GAL22V10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

Commit message: Add files via upload
Parts:
- U5: value 8255 -> 6821
- moved C5 3.14 mm to (135.9, 92.6), turned to 180 degrees
- moved U5 0.11 mm to (142.2, 144.8)
Connections:
- U1 pad 20: /~WE -> /~PIO
- U1 pad 21: /RESET -> /~WE
- U1 pad 23: /~RESET -> /~CLOCK
- U5 pad 1: Net-(U5-Pad1) -> GND
- U5 pad 11: (no net) -> Net-(U5-Pad11)
- U5 pad 12: (no net) -> Net-(U5-Pad12)
- U5 pad 13: (no net) -> Net-(U5-Pad13)
- U5 pad 14: (no net) -> Net-(U5-Pad14)
- U5 pad 15: (no net) -> Net-(U5-Pad15)
- U5 pad 16: Net-(U5-Pad16) -> (no net)
- U5 pad 18: Net-(U5-Pad18) -> (no net)
- U5 pad 19: Net-(U5-Pad19) -> (no net)
- U5 pad 20: Net-(U5-Pad20) -> +5V
- U5 pad 21: Net-(U5-Pad21) -> /~WE
- U5 pad 22: Net-(U5-Pad22) -> /~PIO
- U5 pad 23: Net-(U5-Pad23) -> /PIO
- U5 pad 24: Net-(U5-Pad24) -> /~PIO
- U5 pad 25: Net-(U5-Pad25) -> /~CLOCK
- U5 pad 26: +5V -> /DB7
- U5 pad 27: /DB7 -> /DB6
- U5 pad 28: /DB6 -> /DB5
- U5 pad 29: /DB5 -> /DB4
- U5 pad 30: /DB4 -> /DB3
- U5 pad 31: /DB3 -> /DB2
- U5 pad 32: /DB2 -> /DB1
- U5 pad 33: /DB1 -> /DB0
- U5 pad 34: /DB0 -> /~RESET
- U5 pad 35: /RESET -> /A1
- U5 pad 36: /~WE -> /A0
- U5 pad 5: /~RD -> Net-(U5-Pad5)
- U5 pad 6: /PIO -> Net-(U5-Pad6)
- U5 pad 7: GND -> Net-(U5-Pad7)
- U5 pad 8: /A1 -> Net-(U5-Pad8)
- U5 pad 9: /A0 -> Net-(U5-Pad9)
- U6 pad 10: Net-(U5-Pad23) -> Net-(U5-Pad7)
- U6 pad 11: Net-(U5-Pad24) -> Net-(U5-Pad8)
- U6 pad 12: Net-(U5-Pad25) -> Net-(U5-Pad9)
- U6 pad 17: Net-(U5-Pad10) -> Net-(U5-Pad14)
- U6 pad 18: Net-(U5-Pad16) -> Net-(U5-Pad15)
- U6 pad 19: Net-(U5-Pad4) -> Net-(U5-Pad10)
- U6 pad 20: Net-(U5-Pad3) -> Net-(U5-Pad11)
- U6 pad 5: Net-(U5-Pad18) -> Net-(U5-Pad2)
- U6 pad 6: Net-(U5-Pad19) -> Net-(U5-Pad3)
- U6 pad 7: Net-(U5-Pad20) -> Net-(U5-Pad4)
- U6 pad 8: Net-(U5-Pad21) -> Net-(U5-Pad5)
- U6 pad 9: Net-(U5-Pad22) -> Net-(U5-Pad6)
- U6 pad A4: Net-(U5-Pad2) -> Net-(U5-Pad12)
- U6 pad A5: Net-(U5-Pad1) -> Net-(U5-Pad13)
Routing:
- net /~RD: track 93.8 -> 18.2 mm
- net /DB7: track 181.6 -> 117.9 mm, vias 0 -> 1
- net /RESET: track 59.0 -> 0.00 mm
- net Net-(U5-Pad16): track 54.9 -> 0.00 mm
- net Net-(U5-Pad21): track 45.6 -> 0.00 mm, vias 1 -> 0
- net Net-(U5-Pad22): track 42.0 -> 0.00 mm, vias 1 -> 0
- net Net-(U5-Pad15): track 0.00 -> 40.6 mm, vias 0 -> 1
- net Net-(U5-Pad20): track 40.3 -> 0.00 mm
- net Net-(U5-Pad19): track 39.8 -> 0.00 mm
- net Net-(U5-Pad18): track 38.8 -> 0.00 mm
- net Net-(U5-Pad23): track 38.0 -> 0.00 mm, vias 1 -> 0
- net /~CLOCK: track 0.00 -> 37.5 mm
- net Net-(U5-Pad13): track 0.00 -> 37.0 mm
- net Net-(U5-Pad14): track 0.00 -> 36.8 mm, vias 0 -> 1
- net /PIO: track 59.2 -> 24.0 mm
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Other:
- board text added: "6821"
- board text added: "JR-100_SD Rev2.1"
- board text removed: "8255"
- board text removed: "JR-100_SD Rev1.3"
